File: src/pcb-connector/pcb-connector.kicad_pcb (KiCad board)
At the start: 2 copper layers, 9 x 19 mm, 6 parts, among them J1 Conn_01x02

Commit message: changing pcb connector size
Parts:
- added J2: Conn_01x02, modular-rf-bench-footprints:edge-connector, F.Cu at (145.0, 82.5)
- moved J1 1.00 mm to (150.0, 82.5)
Connections:
- J1 pad 1: unconnected-(J1-Pad1) -> Net-(J1-Pad1)
Routing:
- net GND: vias 16 -> 28
Other:
- outline, holes or cut-outs redrawn
Changed lines of the file:
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@@
   (net 0 "")
   (net 1 "GND")
-  (net 2 "unconnected-(J1-Pad1)")
+  (net 2 "Net-(J1-Pad1)")
   (footprint "modular-rf-bench-footprints:M2-hole" (layer "F.Cu")
     (at 145 90)
@@
   )
   (footprint "modular-rf-bench-footprints:edge-connector" (layer "F.Cu")
-    (at 149 82.5)
+    (at 150 82.5)
     (property "Sheetfile" "pcb-connector.kicad_sch")
     (property "Sheetname" "")
@@
     (fp_line (start 0 -3) (end 0 3) (layer "Cmts.User") (width 0.12))
     (pad "1" smd rect (at -1.5 0) (size 3 1.07801) (layers "F.Cu")
-      (net 2 "unconnected-(J1-Pad1)") (pinfunction "Pin_1") (pintype "passive+no_connect"))
+      (net 2 "Net-(J1-Pad1)") (pinfunction "Pin_1") (pintype "passive"))
     (pad "2" smd rect (at -1.5 -1.739005) (size 3 2) (layers "F.Cu")
       (net 1 "GND") (pinfunction "Pin_2") (pintype "passive"))
@@
     (pad "1" thru_hole circle (at 0 0) (size 3.4 3.4) (drill 2.2) (layers *.Cu *.Mask)
       (net 1 "GND") (pinfunction "1") (pintype "input"))
+  )
+  (footprint "modular-rf-bench-footprints:edge-connector" (layer "F.Cu")
+    (at 145 82.5 180)
+    (property "Sheetfile" "pcb-connector.kicad_sch")
+    (property "Sheetname" "")
+    (attr smd)
+    (fp_text reference "J2" (at -0.5 0 180 unlocked) (layer "F.SilkS") hide
+      (effects (font (size 1 1) (thickness 0.15)))
+    )
+    (fp_text value "Conn_01x02" (at -1.5 1 180 unlocked) (layer "F.Fab") hide
+      (effects (font (size 1 1) (thickness 0.15)))
+    )
+    (fp_text user "EDGE" (at 1 0 270 unlocked) (layer "Cmts.User") hide
+      (effects (font (size 1 1) (thickness 0.15)))
+    )
+    (fp_text user "${REFERENCE}" (at -1 2 180 unlocked) (layer "F.Fab") hide
+      (effects (font (size 1 1) (thickness 0.15)))
+    )
+    (fp_poly (pts
+        (xy 0 2)
+        (xy -3 2)
+        (xy -3 -2)
+        (xy 0 -2)
+      ) (layer "F.Mask") (width 0) (fill solid))
+    (fp_line (start 0 -3) (end 0 3) (layer "Cmts.User") (width 0.1))
+    (pad "1" smd rect (at -1.5 0 180) (size 3 1.07801) (layers "F.Cu")
+      (net 2 "Net-(J1-Pad1)") (pinfunction "Pin_1") (pintype "passive"))
+    (pad "2" smd rect (at -1.5 -1.739005 180) (size 3 2) (layers "F.Cu")
+      (net 1 "GND") (pinfunction "Pin_2") (pintype "passive"))
+    (pad "2" smd rect (at -1.5 1.739005 180) (size 3 2) (layers "F.Cu")
+      (net 1 "GND") (pinfunction "Pin_2") (pintype "passive"))
   )
   (footprint "modular-rf-bench-footprints:M2-hole" (layer "F.Cu")
@@
   )
   (gr_line (start 145 73) (end 150 73) (layer "Edge.Cuts") (width 0.1))
-  (gr_line (start 146 79.5) (end 146 85.5) (layer "Edge.Cuts") (width 0.1))
+  (gr_line (start 145 79.5) (end 145 85.5) (layer "Edge.Cuts") (width 0.1))
   (gr_line (start 145 92) (end 150 92) (layer "Edge.Cuts") (width 0.1))
-  (gr_line (start 150 77) (end 149 79.5) (layer "Edge.Cuts") (width 0.1))
-  (gr_line (start 146 85.5) (end 145 88) (layer "Edge.Cuts") (width 0.1))
+  (gr_line (start 150 77) (end 150 79.5) (layer "Edge.Cuts") (width 0.1))
+  (gr_line (start 145 85.5) (end 145 88) (layer "Edge.Cuts") (width 0.1))
   (gr_arc (start 150 88) (mid 152 90) (end 150 92) (layer "Edge.Cuts") (width 0.1))
   (gr_arc (start 145 77) (mid 143 75) (end 145 73) (layer "Edge.Cuts") (width 0.1))
-  (gr_line (start 149 85.5) (end 150 88) (layer "Edge.Cuts") (width 0.1))
-  (gr_line (start 149 79.5) (end 149 85.5) (layer "Edge.Cuts") (width 0.1))
-  (gr_line (start 145 77) (end 146 79.5) (layer "Edge.Cuts") (width 0.1))
+  (gr_line (start 150 85.5) (end 150 88) (layer "Edge.Cuts") (width 0.1))
+  (gr_line (start 150 79.5) (end 150 85.5) (layer "Edge.Cuts") (width 0.1))
+  (gr_line (start 145 77) (end 145 79.5) (layer "Edge.Cuts") (width 0.1))
   (gr_arc (start 150 73) (mid 152 75) (end 150 77) (layer "Edge.Cuts") (width 0.1))
   (gr_arc (start 145 92) (mid 143 90) (end 145 88) (layer "Edge.Cuts") (width 0.1))
   (via (at 148.5 81) (size 0.8) (drill 0.4) (layers "F.Cu" "B.Cu") (net 1))
+  (via (at 149 80.5) (size 0.8) (drill 0.4) (layers "F.Cu" "B.Cu") (net 1))
   (via (at 147.5 85) (size 0.8) (drill 0.4) (layers "F.Cu" "B.Cu") (net 1))
   (via (at 147 80.5) (size 0.8) (drill 0.4) (layers "F.Cu" "B.Cu") (net 1))
+  (via (at 149 84.5) (size 0.8) (drill 0.4) (layers "F.Cu" "B.Cu") (net 1))
+  (via (at 146 80.5) (size 0.8) (drill 0.4) (layers "F.Cu" "B.Cu") (net 1))
   (via (at 146.5 84) (size 0.8) (drill 0.4) (layers "F.Cu" "B.Cu") (net 1))
   (via (at 148 80.5) (size 0.8) (drill 0.4) (layers "F.Cu" "B.Cu") (net 1))
+  (via (at 149.5 81) (size 0.8) (drill 0.4) (layers "F.Cu" "B.Cu") (net 1))
   (via (at 148 84.5) (size 0.8) (drill 0.4) (layers "F.Cu" "B.Cu") (net 1))
   (via (at 148.5 84) (size 0.8) (drill 0.4) (layers "F.Cu" "B.Cu") (net 1))
+  (via (at 149.5 85) (size 0.8) (drill 0.4) (layers "F.Cu" "B.Cu") (net 1))
   (via (at 147.5 84) (size 0.8) (drill 0.4) (layers "F.Cu" "B.Cu") (net 1))
   (via (at 146.5 81) (size 0.8) (drill 0.4) (layers "F.Cu" "B.Cu") (net 1))
+  (via (at 146 84.5) (size 0.8) (drill 0.4) (layers "F.Cu" "B.Cu") (net 1))
   (via (at 147 84.5) (size 0.8) (drill 0.4) (layers "F.Cu" "B.Cu") (net 1))
   (via (at 146.5 80) (size 0.8) (drill 0.4) (layers "F.Cu" "B.Cu") (net 1))
@@
   (via (at 148.5 85) (size 0.8) (drill 0.4) (layers "F.Cu" "B.Cu") (net 1))
   (via (at 147.5 81) (size 0.8) (drill 0.4) (layers "F.Cu" "B.Cu") (net 1))
+  (via (at 145.5 80) (size 0.8) (drill 0.4) (layers "F.Cu" "B.Cu") (net 1))
   (via (at 146.5 85) (size 0.8) (drill 0.4) (layers "F.Cu" "B.Cu") (net 1))
+  (via (at 145.5 84) (size 0.8) (drill 0.4) (layers "F.Cu" "B.Cu") (net 1))
+  (via (at 149.5 80) (size 0.8) (drill 0.4) (layers "F.Cu" "B.Cu") (net 1))
+  (via (at 145.5 81) (size 0.8) (drill 0.4) (layers "F.Cu" "B.Cu") (net 1))
+  (via (at 149.5 84) (size 0.8) (drill 0.4) (layers "F.Cu" "B.Cu") (net 1))
+  (via (at 145.5 85) (size 0.8) (drill 0.4) (layers "F.Cu" "B.Cu") (net 1))
   (zone (net 1) (net_name "GND") (layers F&B.Cu) (hatch edge 0.508)
     (connect_pads yes (clearance 0.2))
