File: src/001-base/base.kicad_pcb (KiCad board)
At the start: 2 copper layers, 99 x 99 mm, 397 parts

Commit message: changing base
Other:
- board text added: "001"
- board text removed: "MODULAR RF BENCH HALIDELABS"
Changed lines of the file:
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@@
   )
   (paper "A4")
+  (title_block
+    (title "001 Base")
+    (date "2022-01-27")
+    (rev "1")
+    (company "Halidelabs")
+    (comment 1 "contact@halidelabs.eu")
+  )
   (layers
     (0 "F.Cu" signal "Górna sygnałowa")
     (31 "B.Cu" signal "Dolna sygnałowa")
-    (32 "B.Adhes" user "Dolna kleju")
-    (33 "F.Adhes" user "Górna kleju")
-    (34 "B.Paste" user "Dolna pasty")
-    (35 "F.Paste" user "Górna pasty")
     (36 "B.SilkS" user "Dolna opisowa")
-    (37 "F.SilkS" user "Górna opisowa")
     (38 "B.Mask" user "Dolna sodermaski")
     (39 "F.Mask" user "Górna soldermaski")
-    (40 "Dwgs.User" user "Rysunkowa użytkownika")
-    (41 "Cmts.User" user "Komentarzy użytkownika")
-    (42 "Eco1.User" user "Inżynieryjna 1")
-    (43 "Eco2.User" user "Inżynieryjna 2")
     (44 "Edge.Cuts" user "Krawędziowa")
     (45 "Margin" user "Marginesu")
     (46 "B.CrtYd" user "Dolne pola zajętości")
     (47 "F.CrtYd" user "Górne pola zajętości")
-    (48 "B.Fab" user "Dolna produkcyjna")
-    (49 "F.Fab" user "Górna produkcyjna")
-    (50 "User.1" user "Użytkownika 1")
-    (51 "User.2" user "Użytkownika 2")
-    (52 "User.3" user "Użytkownika 3")
-    (53 "User.4" user "Użytkownika 4")
-    (54 "User.5" user "Użytkownika 5")
-    (55 "User.6" user "Użytkownika 6")
-    (56 "User.7" user "Użytkownika 7")
-    (57 "User.8" user "Użytkownika 8")
-    (58 "User.9" user "Użytkownika 9")
   )
   (setup
     (stackup
-      (layer "F.SilkS" (type "Top Silk Screen"))
-      (layer "F.Paste" (type "Top Solder Paste"))
-      (layer "F.Mask" (type "Top Solder Mask") (thickness 0.01))
+      (layer "F.Mask" (type "Top Solder Mask") (color "Black") (thickness 0.01))
       (layer "F.Cu" (type "copper") (thickness 0.035))
       (layer "dielectric 1" (type "core") (thickness 1.51) (material "FR4") (epsilon_r 4.5) (loss_tangent 0.02))
       (layer "B.Cu" (type "copper") (thickness 0.035))
-      (layer "B.Mask" (type "Bottom Solder Mask") (thickness 0.01))
-      (layer "B.Paste" (type "Bottom Solder Paste"))
-      (layer "B.SilkS" (type "Bottom Silk Screen"))
-      (copper_finish "None")
+      (layer "B.Mask" (type "Bottom Solder Mask") (color "Black") (thickness 0.01))
+      (layer "B.SilkS" (type "Bottom Silk Screen") (color "White"))
+      (copper_finish "Immersion gold")
       (dielectric_constraints no)
     )
     (pad_to_mask_clearance 0)
     (pcbplotparams
-      (layerselection 0x00010f0_ffffffff)
+      (layerselection 0x00010d0_ffffffff)
       (disableapertmacros false)
       (usegerberextensions false)
@@
   (gr_arc (start 99 146) (mid 97.585786 145.414214) (end 97 144) (layer "Edge.Cuts") (width 0.1))
   (gr_line (start 99 47) (end 194 47) (layer "Edge.Cuts") (width 0.1))
-  (gr_text "MODULAR\nRF BENCH\n\n\nHALIDELABS" (at 106.5 136.5) (layer "B.Cu")
+  (gr_text "001" (at 106.5 136.5) (layer "B.SilkS")
     (effects (font (size 1 1) (thickness 0.15)) (justify mirror))
   )
@@
     )
   )
-  (zone (net 0) (net_name "") (layers *.Mask) (name "GND") (hatch edge 0.508)
+  (zone (net 0) (net_name "") (layer "B.Mask") (name "GND") (hatch edge 0.508)
     (connect_pads yes (clearance 0.3))
     (min_thickness 0.254) (filled_areas_thickness no)
@@
     (polygon
       (pts
+        (xy 196 135.5)
+        (xy 97 135.5)
+        (xy 97 47)
+        (xy 196 47)
+      )
+    )
+  )
+  (zone (net 0) (net_name "") (layer "B.Mask") (name "GND") (hatch edge 0.508)
+    (connect_pads yes (clearance 0.3))
+    (min_thickness 0.254) (filled_areas_thickness no)
+    (fill yes (thermal_gap 0.3) (thermal_bridge_width 0.3))
+    (polygon
+      (pts
+        (xy 105 137.5)
+        (xy 97 137.5)
+        (xy 97 135.5)
+        (xy 105 135.5)
+      )
+    )
+  )
+  (zone (net 0) (net_name "") (layer "B.Mask") (hatch edge 0.508)
+    (connect_pads (clearance 0.26))
+    (min_thickness 0.254) (filled_areas_thickness no)
+    (fill yes (thermal_gap 0.508) (thermal_bridge_width 0.508))
+    (polygon
+      (pts
         (xy 196 146)
         (xy 97 146)
+        (xy 97 137.5)
+        (xy 196 137.5)
+      )
+    )
+  )
+  (zone (net 0) (net_name "") (layer "B.Mask") (name "GND") (hatch edge 0.508)
+    (connect_pads yes (clearance 0.3))
+    (min_thickness 0.254) (filled_areas_thickness no)
+    (fill yes (thermal_gap 0.3) (thermal_bridge_width 0.3))
+    (polygon
+      (pts
+        (xy 196 137.5)
+        (xy 108 137.5)
+        (xy 108 135.5)
+        (xy 196 135.5)
+      )
+    )
+  )
+  (zone (net 0) (net_name "") (layer "F.Mask") (name "GND") (hatch edge 0.508)
+    (connect_pads yes (clearance 0.3))
+    (min_thickness 0.254) (filled_areas_thickness no)
+    (fill yes (thermal_gap 0.3) (thermal_bridge_width 0.3))
+    (polygon
+      (pts
+        (xy 196 145.967)
+        (xy 97 145.967)
         (xy 97 47)
         (xy 196 47)
