File: src/002-sma-connector/sma-connector.kicad_pcb (KiCad board)
At the start: 2 copper layers, 15 x 20 mm, 7 parts, among them J1 SMA, J2 EDGE CONN

Commit message: changing sma connector pcb
Routing:
- net GND: vias 116 -> 39
Other:
- board text added: "002"
