File: src/002-sma-connector/sma-connector.kicad_sch (KiCad schematic)
At the start: 6 parts, among them J1 SMA, J2 EDGE CONN

Commit message: changing sma connector pcb
Other:
- company: (none) -> Halidelabs
- title: (none) -> 002-SMA Connector
Changed lines of the file:
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@@
 (kicad_sch (version 20211123) (generator eeschema)
   (paper "A4")
+  (title_block
+    (title "002-SMA Connector")
+    (date "2022-01-27")
+    (rev "1")
+    (company "Halidelabs")
+    (comment 1 "contact@halidelabs.eu")
+  )
   (wire (pts (xy 124.46 125.73) (xy 124.46 127))
     (stroke (width 0) (type default) (color 0 0 0 0))
