File: src/003-pcb-connector/pcb-connector.kicad_sch (KiCad schematic)
At the start: 6 parts, among them J1 Conn_01x02, J2 Conn_01x02

Commit message: changing pcb connector
Parts:
- J1, J2: value Conn_01x02 -> CONN
Other:
- company: (none) -> Halidelabs
- title: (none) -> 003-PCB Connector
Changed lines of the file:
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@@
 (kicad_sch (version 20211123) (generator eeschema)
   (paper "A4")
+  (title_block
+    (title "003-PCB Connector")
+    (date "2022-01-27")
+    (rev "1")
+    (company "Halidelabs")
+    (comment 1 "contact@halidelabs.eu")
+  )
   (junction (at 142.24 93.98) (diameter 0) (color 0 0 0 0)
   )
@@
       (effects (font (size 1.27 1.27)) (justify left))
     )
-    (property "Value" "Conn_01x02" (id 1) (at 151.13 93.9799 0)
+    (property "Value" "CONN" (id 1) (at 151.13 93.9799 0)
       (effects (font (size 1.27 1.27)) (justify left))
     )
@@
     (in_bom yes) (on_board yes)
     (property "Reference" "J2" (id 0) (at 132.08 91.44 0))
-    (property "Value" "Conn_01x02" (id 1) (at 128.27 93.98 0))
+    (property "Value" "CONN" (id 1) (at 130.81 93.98 0))
     (property "Footprint" "modular-rf-bench-footprints:edge-connector" (id 2) (at 135.89 91.44 0)
       (effects (font (size 1.27 1.27)) hide)
@@
     )
     (path "/7c5779b7-3d70-4446-a23a-f4cf05b5eb95"
-      (reference "J1") (unit 1) (value "Conn_01x02") (footprint "modular-rf-bench-footprints:edge-connector")
+      (reference "J1") (unit 1) (value "CONN") (footprint "modular-rf-bench-footprints:edge-connector")
     )
     (path "/d0111086-5d68-4ab0-b707-7da6b263c90b"
-      (reference "J2") (unit 1) (value "Conn_01x02") (footprint "modular-rf-bench-footprints:edge-connector")
-    )
-  )
+      (reference "J2") (unit 1) (value "CONN") (footprint "modular-rf-bench-footprints:edge-connector")
+    )
+  )
