File: src/004-pcb-turn-45/pcb-turn-45.kicad_sch (KiCad schematic)
At the start: 6 parts, among them J1 CONN, J2 CONN

Commit message: adding filter pcb and load
Other:
- company: (none) -> Halidelabs
- title: (none) -> 004 PCB 45 Turn
Changed lines of the file:
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@@
 (kicad_sch (version 20211123) (generator eeschema)
   (paper "A4")
+  (title_block
+    (title "004 PCB 45 Turn")
+    (date "2022-01-28")
+    (rev "1")
+    (company "Halidelabs")
+    (comment 1 "contact@halidelabs.eu")
+  )
   (junction (at 144.78 95.25) (diameter 0) (color 0 0 0 0)
   )
