File: src/005-pcb-connector-x2/pcb-connector-x2.kicad_pcb (KiCad board)
At the start: 2 copper layers, 24 x 24 mm, 11 parts, among them J1 CONN, J2 CONN, J3 CONN, J4 CONN

Commit message: adding filter pcb and load
Parts:
- added G***: LOGO, LOGO, B.Cu at (142.8, 102.2)
- moved H1 45.0 mm to (155.0, 100.0)
- moved H2 45.0 mm to (140.0, 105.0)
- moved H3 45.0 mm to (140.0, 100.0)
- moved H4 45.0 mm to (135.0, 100.0)
- moved H5 45.0 mm to (155.0, 105.0)
- moved H6 45.0 mm to (135.0, 85.0)
- moved H7 45.0 mm to (140.0, 85.0)
- moved J1 45.0 mm to (147.5, 100.0)
- moved J2 45.0 mm to (140.0, 92.5)
- moved J3 45.0 mm to (147.5, 105.0)
- moved J4 45.0 mm to (135.0, 92.5)
Routing:
- added copper zone on B.Cu, net GND
- added copper zone on F.Cu, net GND
Other:
- board text added: "005"
