File: src/014-base-power-board/014-base-power-board.kicad_sch (KiCad schematic)
At the start: 16 parts, among them J1 GND, J10 V4, J2 GND, J3 V1, J4 V1, J5 V2, J6 V2, J7 V3, J8 V3, J9 V4

Commit message: Adding 014-base-power-board
Parts:
- J10, J2, J4, J6, J8: footprint Connector_PinHeader_2.54mm:PinHeader_1x08_P2.54mm_Vertical_SMD_Pin1Left -> Connector_PinHeader_2.54mm:PinHeader_1x06_P2.54mm_Vertical_SMD_Pin1Left; symbol Connector_Generic:Conn_01x08 -> Connector_Generic:Conn_01x06
Connections:
- net GND: no longer J2.7 (Pin_7), J2.8 (Pin_8)
- net at J7.1 (Pin_1), J8.1 (Pin_1), J8.2 (Pin_2)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: no longer J8.7 (Pin_7), J8.8 (Pin_8)
- net at J3.1 (Pin_1), J4.1 (Pin_1), J4.2 (Pin_2)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: no longer J4.7 (Pin_7), J4.8 (Pin_8)
- net at J5.1 (Pin_1), J6.1 (Pin_1), J6.2 (Pin_2)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: no longer J6.7 (Pin_7), J6.8 (Pin_8)
- net at J10.1 (Pin_1), J10.2 (Pin_2), J10.3 (Pin_3)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: no longer J10.7 (Pin_7), J10.8 (Pin_8)
